Commit message: Update ellie_bot.xacro

File: urdf/ellie_bot.xacro (robot description, xacro)
@@ -177,10 +177,10 @@
     <parent link="chassis"/>
 </joint>
-  <joint name="camera_rgb_joint" type="fixed">
+  <joint name="camera_rgbd_joint" type="fixed">
     <origin xyz="0 -0.012 0" rpy="0 0 0" />
     <parent link="camera" />
-    <child link="camera_rgb_frame" />
+    <child link="camera_rgbd_frame" />
   </joint>
-  <link name="camera_rgb_frame">
+  <link name="camera_rgbd_frame">
     <inertial>
       <mass value="0.001" />

Commit message: Update ellie_bot.xacro

File: urdf/ellie_bot.xacro (robot description, xacro)
@@ -178,5 +178,5 @@
 </joint>
   <joint name="camera_rgbd_joint" type="fixed">
-    <origin xyz="0 -0.012 0" rpy="0 0 0" />
+    <origin xyz="0 0 0" rpy="-1.5707 0 -1.5707" />
     <parent link="camera" />
     <child link="camera_rgbd_frame" />
